File: doc/eagle/cubey_v3.sch (EAGLE design)
At the start: 24 parts, among them K1 PIN20X2

Commit message: Update v3 board layout, with cutout for RPi camera, remove of v2 designs
Other:
- note removed: "Checked by:"
- note removed: "Drawn by:"
- note removed: "FLYFISH TECHNOLOGIES d.o.o."
- note removed: "Ivan Zilic"
- note removed: "v0.1"
- moved on the sheet: BACK, BTN, C2, C3, C4, C5, C6, C8, DOWN, FRONT, JP1, JP16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
